Commit message: ya hay pato en gazebo y rviz

File: install/urdf_description/share/urdf_description/urdf/go_bdx.urdf.xacro (robot description, xacro)
@@ -2,5 +2,5 @@
 <robot name="bdx" xmlns:xacro="http://www.ros.org/wiki/xacro">
   <material name="silver">
-    <color rgba="0.700 0.700 0.700 1.000"/>
+    <color rgba="1.0 1.0 0.0 1.0"/>
   </material>
   <link name="trunk">
@@ -138,5 +138,5 @@
       <origin rpy="0 0 0" xyz="0 0 0"/>
       <geometry>
-        <mesh filename="package://urdf_description/meshes/pelvis.stl" scale=".001 .001 .001"/>
+        <mesh filename="file://$(find urdf_description)/meshes/pelvis.stl" scale=".001 .001 .001"/>
       </geometry>
       <material name="silver"/>
@@ -145,5 +145,5 @@
       <origin rpy="0 0 0" xyz="0 0 0"/>
       <geometry>
-        <mesh filename="package://urdf_description/meshes/pelvis.stl" scale=".001 .001 .001"/>
+        <mesh filename="file://$(find urdf_description)/meshes/pelvis.stl" scale=".001 .001 .001"/>
       </geometry>
     </collision>
@@ -171,5 +171,5 @@
       <origin rpy="0 0 0" xyz="0.057251 -0.103809 -0.081036"/>
       <geometry>
-        <mesh filename="package://urdf_description/meshes/left_foot.stl" scale=".001 .001 .001"/>
+        <mesh filename="file://$(find urdf_description)/meshes/left_foot.stl" scale=".001 .001 .001"/>
       </geometry>
       <material name="silver"/>
@@ -178,5 +178,5 @@
       <origin rpy="0 0 0" xyz="0.057251 -0.103809 -0.081036"/>
       <geometry>
-        <mesh filename="package://urdf_description/meshes/left_foot.stl" scale=".001 .001 .001"/>
+        <mesh filename="file://$(find urdf_description)/meshes/left_foot.stl" scale=".001 .001 .001"/>
       </geometry>
     </collision>
@@ -191,5 +191,5 @@
       <origin rpy="0 0 0" xyz="0.102251 -0.119009 -0.211036"/>
       <geometry>
-        <mesh filename="package://urdf_description/meshes/left_shin.stl" scale=".001 .001 .001"/>
+        <mesh filename="file://$(find urdf_description)/meshes/left_shin.stl" scale=".001 .001 .001"/>
       </geometry>
       <material name="silver"/>
@@ -198,5 +198,5 @@
       <origin rpy="0 0 0" xyz="0.102251 -0.119009 -0.211036"/>
       <geometry>
-        <mesh filename="package://urdf_description/meshes/left_shin.stl" scale=".001 .001 .001"/>
+        <mesh filename="file://$(find urdf_description)/meshes/left_shin.stl" scale=".001 .001 .001"/>
       </geometry>
     </collision>
@@ -211,5 +211,5 @@
       <origin rpy="0 0 0" xyz="0.022945 -0.119009 -0.288744"/>
       <geometry>
-        <mesh filename="package://urdf_description/meshes/left_thigh.stl" scale=".001 .001 .001"/>
+        <mesh filename="file://$(find urdf_description)/meshes/left_thigh.stl" scale=".001 .001 .001"/>
       </geometry>
       <material name="silver"/>
@@ -218,5 +218,5 @@
       <origin rpy="0 0 0" xyz="0.022945 -0.119009 -0.288744"/>
       <geometry>
-        <mesh filename="package://urdf_description/meshes/left_thigh.stl" scale=".001 .001 .001"/>
+        <mesh filename="file://$(find urdf_description)/meshes/left_thigh.stl" scale=".001 .001 .001"/>
       </geometry>
     </collision>
@@ -231,5 +231,5 @@
       <origin rpy="0 0 0" xyz="0.040411 -0.049408 -0.287959"/>
       <geometry>
-        <mesh filename="package://urdf_description/meshes/left_hip.stl" scale=".001 .001 .001"/>
+        <mesh filename="file://$(find urdf_description)/meshes/left_hip.stl" scale=".001 .001 .001"/>
       </geometry>
       <material name="silver"/>
@@ -238,5 +238,5 @@
       <origin rpy="0 0 0" xyz="0.040411 -0.049408 -0.287959"/>
       <geometry>
-        <mesh filename="package://urdf_description/meshes/left_hip.stl" scale=".001 .001 .001"/>
+        <mesh filename="file://$(find urdf_description)/meshes/left_hip.stl" scale=".001 .001 .001"/>
       </geometry>
     </collision>
@@ -251,5 +251,5 @@
       <origin rpy="0 0 0" xyz="0.033111 -0.046658 -0.363959"/>
       <geometry>
-        <mesh filename="package://urdf_description/meshes/left_hip_rotation.stl" scale=".001 .001 .001"/>
+        <mesh filename="file://$(find urdf_description)/meshes/left_hip_rotation.stl" scale=".001 .001 .001"/>
       </geometry>
       <material name="silver"/>
@@ -258,5 +258,5 @@
       <origin rpy="0 0 0" xyz="0.033111 -0.046658 -0.363959"/>
       <geometry>
-        <mesh filename="package://urdf_description/meshes/left_hip_rotation.stl" scale=".001 .001 .001"/>
+        <mesh filename="file://$(find urdf_description)/meshes/left_hip_rotation.stl" scale=".001 .001 .001"/>
       </geometry>
     </collision>
@@ -284,5 +284,5 @@
       <origin rpy="0 0 0" xyz="0.057251 0.103809 -0.081036"/>
       <geometry>
-        <mesh filename="package://urdf_description/meshes/right_foot.stl" scale=".001 .001 .001"/>
+        <mesh filename="file://$(find urdf_description)/meshes/right_foot.stl" scale=".001 .001 .001"/>
       </geometry>
       <material name="silver"/>
@@ -291,5 +291,5 @@
       <origin rpy="0 0 0" xyz="0.057251 0.103809 -0.081036"/>
       <geometry>
-        <mesh filename="package://urdf_description/meshes/right_foot.stl" scale=".001 .001 .001"/>
+        <mesh filename="file://$(find urdf_description)/meshes/right_foot.stl" scale=".001 .001 .001"/>
       </geometry>
     </collision>
@@ -304,5 +304,5 @@
       <origin rpy="0 0 0" xyz="0.102251 0.119009 -0.211036"/>
       <geometry>
-        <mesh filename="package://urdf_description/meshes/right_shin.stl" scale=".001 .001 .001"/>
+        <mesh filename="file://$(find urdf_description)/meshes/right_shin.stl" scale=".001 .001 .001"/>
       </geometry>
       <material name="silver"/>
@@ -311,5 +311,5 @@
       <origin rpy="0 0 0" xyz="0.102251 0.119009 -0.211036"/>
       <geometry>
-        <mesh filename="package://urdf_description/meshes/right_shin.stl" scale=".001 .001 .001"/>
+        <mesh filename="file://$(find urdf_description)/meshes/right_shin.stl" scale=".001 .001 .001"/>
       </geometry>
     </collision>
@@ -324,5 +324,5 @@
       <origin rpy="0 0 0" xyz="0.022945 0.119009 -0.288744"/>
       <geometry>
-        <mesh filename="package://urdf_description/meshes/right_thigh.stl" scale=".001 .001 .001"/>
+        <mesh filename="file://$(find urdf_description)/meshes/right_thigh.stl" scale=".001 .001 .001"/>
       </geometry>
       <material name="silver"/>
@@ -331,5 +331,5 @@
       <origin rpy="0 0 0" xyz="0.022945 0.119009 -0.288744"/>
       <geometry>
-        <mesh filename="package://urdf_description/meshes/right_thigh.stl" scale=".001 .001 .001"/>
+        <mesh filename="file://$(find urdf_description)/meshes/right_thigh.stl" scale=".001 .001 .001"/>
       </geometry>
     </collision>
@@ -344,5 +344,5 @@
       <origin rpy="0 0 0" xyz="0.040411 0.049408 -0.287959"/>
       <geometry>
-        <mesh filename="package://urdf_description/meshes/right_hip.stl" scale=".001 .001 .001"/>
+        <mesh filename="file://$(find urdf_description)/meshes/right_hip.stl" scale=".001 .001 .001"/>
       </geometry>
       <material name="silver"/>
@@ -351,5 +351,5 @@
       <origin rpy="0 0 0" xyz="0.040411 0.049408 -0.287959"/>
       <geometry>
-        <mesh filename="package://urdf_description/meshes/right_hip.stl" scale=".001 .001 .001"/>
+        <mesh filename="file://$(find urdf_description)/meshes/right_hip.stl" scale=".001 .001 .001"/>
       </geometry>
     </collision>
@@ -364,5 +364,5 @@
       <origin rpy="0 0 0" xyz="0.033111 0.046658 -0.363959"/>
       <geometry>
-        <mesh filename="package://urdf_description/meshes/right_hip_rotation.stl" scale=".001 .001 .001"/>
+        <mesh filename="file://$(find urdf_description)/meshes/right_hip_rotation.stl" scale=".001 .001 .001"/>
       </geometry>
       <material name="silver"/>
@@ -371,5 +371,5 @@
       <origin rpy="0 0 0" xyz="0.033111 0.046658 -0.363959"/>
       <geometry>
-        <mesh filename="package://urdf_description/meshes/right_hip_rotation.stl" scale=".001 .001 .001"/>
+        <mesh filename="file://$(find urdf_description)/meshes/right_hip_rotation.stl" scale=".001 .001 .001"/>
       </geometry>
     </collision>
@@ -384,5 +384,5 @@
       <origin rpy="0 0 0" xyz="0.135142 0.06885 -0.563402"/>
       <geometry>
-        <mesh filename="package://urdf_description/meshes/ear_right.stl" scale=".001 .001 .001"/>
+        <mesh filename="file://$(find urdf_description)/meshes/ear_right.stl" scale=".001 .001 .001"/>
       </geometry>
       <material name="silver"/>
@@ -391,5 +391,5 @@
       <origin rpy="0 0 0" xyz="0.135142 0.06885 -0.563402"/>
       <geometry>
-        <mesh filename="package://urdf_description/meshes/ear_right.stl" scale=".001 .001 .001"/>
+        <mesh filename="file://$(find urdf_description)/meshes/ear_right.stl" scale=".001 .001 .001"/>
       </geometry>
     </collision>
@@ -404,5 +404,5 @@
       <origin rpy="0 0 0" xyz="0.135142 -0.06915 -0.563402"/>
       <geometry>
-        <mesh filename="package://urdf_description/meshes/ear_left.stl" scale=".001 .001 .001"/>
+        <mesh filename="file://$(find urdf_description)/meshes/ear_left.stl" scale=".001 .001 .001"/>
       </geometry>
       <material name="silver"/>
@@ -411,5 +411,5 @@
       <origin rpy="0 0 0" xyz="0.135142 -0.06915 -0.563402"/>
       <geometry>
-        <mesh filename="package://urdf_description/meshes/ear_left.stl" scale=".001 .001 .001"/>
+        <mesh filename="file://$(find urdf_description)/meshes/ear_left.stl" scale=".001 .001 .001"/>
       </geometry>
     </collision>
@@ -437,5 +437,5 @@
       <origin rpy="0 0 0" xyz="-0.031508 -0.00085 -0.562171"/>
       <geometry>
-        <mesh filename="package://urdf_description/meshes/head_body_roll.stl" scale=".001 .001 .001"/>
+        <mesh filename="file://$(find urdf_description)/meshes/head_body_roll.stl" scale=".001 .001 .001"/>
       </geometry>
       <material name="silver"/>
@@ -444,5 +444,5 @@
       <origin rpy="0 0 0" xyz="-0.031508 -0.00085 -0.562171"/>
       <geometry>
-        <mesh filename="package://urdf_description/meshes/head_body_roll.stl" scale=".001 .001 .001"/>
+        <mesh filename="file://$(find urdf_description)/meshes/head_body_roll.stl" scale=".001 .001 .001"/>
       </geometry>
     </collision>
@@ -457,5 +457,5 @@
       <origin rpy="0 0 0" xyz="0.008384 -0.00085 -0.535021"/>
       <geometry>
-        <mesh filename="package://urdf_description/meshes/head_body_yaw.stl" scale=".001 .001 .001"/>
+        <mesh filename="file://$(find urdf_description)/meshes/head_body_yaw.stl" scale=".001 .001 .001"/>
       </geometry>
       <material name="silver"/>
@@ -464,5 +464,5 @@
       <origin rpy="0 0 0" xyz="0.008384 -0.00085 -0.535021"/>
       <geometry>
-        <mesh filename="package://urdf_description/meshes/head_body_yaw.stl" scale=".001 .001 .001"/>
+        <mesh filename="file://$(find urdf_description)/meshes/head_body_yaw.stl" scale=".001 .001 .001"/>
       </geometry>
     </collision>
@@ -477,5 +477,5 @@
       <origin rpy="0 0 0" xyz="0.008683 -0.00015 -0.506051"/>
       <geometry>
-        <mesh filename="package://urdf_description/meshes/head_body_pitch.stl" scale=".001 .001 .001"/>
+        <mesh filename="file://$(find urdf_description)/meshes/head_body_pitch.stl" scale=".001 .001 .001"/>
       </geometry>
       <material name="silver"/>
@@ -484,5 +484,5 @@
       <origin rpy="0 0 0" xyz="0.008683 -0.00015 -0.506051"/>
       <geometry>
-        <mesh filename="package://urdf_description/meshes/head_body_pitch.stl" scale=".001 .001 .001"/>
+        <mesh filename="file://$(find urdf_description)/meshes/head_body_pitch.stl" scale=".001 .001 .001"/>
       </geometry>
     </collision>
@@ -497,5 +497,5 @@
       <origin rpy="0 0 0" xyz="-0.056339 -0.0119 -0.395171"/>
       <geometry>
-        <mesh filename="package://urdf_description/meshes/neck.stl" scale=".001 .001 .001"/>
+        <mesh filename="file://$(find urdf_description)/meshes/neck.stl" scale=".001 .001 .001"/>
       </geometry>
       <material name="silver"/>
@@ -504,5 +504,5 @@
       <origin rpy="0 0 0" xyz="-0.056339 -0.0119 -0.395171"/>
       <geometry>
-        <mesh filename="package://urdf_description/meshes/neck.stl" scale=".001 .001 .001"/>
+        <mesh filename="file://$(find urdf_description)/meshes/neck.stl" scale=".001 .001 .001"/>
       </geometry>
     </collision>

File: src/urdf_description/urdf/go_bdx.urdf.xacro (robot description, xacro)
@@ -1,6 +1,6 @@
 <?xml version="1.0" ?>
-<robot name="bdx">
+<robot name="bdx" xmlns:xacro="http://www.ros.org/wiki/xacro">
   <material name="silver">
-    <color rgba="0.700 0.700 0.700 1.000"/>
+    <color rgba="1.0 1.0 0.0 1.0"/>
   </material>
   <link name="trunk">
