Commit message: parado con static

File: src/urdf_description/urdf/go_bdx.urdf.xacro (robot description, xacro)
@@ -6,7 +6,9 @@
   <link name="trunk">
     <inertial>
-      <origin xyz="0 0 0" rpy="0 0 0" />
-      <mass value="1e-9" />
-      <inertia ixx="0" ixy="0" ixz="0" iyy="0" iyz="0" izz="0" />
+      <origin xyz="0 0 0" rpy="0 0 0"/>
+      <mass value="1.0"/>
+      <inertia
+        ixx="0.005" ixy="0.0" ixz="0.0"
+        iyy="0.005" iyz="0.0" izz="0.005"/>
     </inertial>
   </link>
@@ -151,7 +153,9 @@
   <link name="left_foot">
     <inertial>
-      <origin xyz="0 0 0" rpy="0 0 0" />
-      <mass value="1e-9" />
-      <inertia ixx="0" ixy="0" ixz="0" iyy="0" iyz="0" izz="0" />
+      <origin xyz="0 0 0" rpy="0 0 0"/>
+      <mass value="0.5"/>
+      <inertia
+        ixx="0.0002" ixy="0.0" ixz="0.0"
+        iyy="0.0002" iyz="0.0" izz="0.0002"/>
     </inertial>
   </link>
@@ -264,7 +268,9 @@
   <link name="right_foot">
     <inertial>
-      <origin xyz="0 0 0" rpy="0 0 0" />
-      <mass value="1e-9" />
-      <inertia ixx="0" ixy="0" ixz="0" iyy="0" iyz="0" izz="0" />
+      <origin xyz="0 0 0" rpy="0 0 0"/>
+      <mass value="0.5"/>
+      <inertia
+        ixx="0.0002" ixy="0.0" ixz="0.0"
+        iyy="0.0002" iyz="0.0" izz="0.0002"/>
     </inertial>
   </link>
@@ -729,7 +735,24 @@
   <gazebo>
     <plugin filename="libgazebo_ros2_control.so" name="gazebo_ros2_control">
-      <!-- Asegúrate de apuntar al paquete correcto -->
       <parameters>$(find urdf_description)/config/controllers.yaml</parameters>
     </plugin>
   </gazebo>
+  <gazebo reference="left_foot">
+    <mu1>1.5</mu1>  <!-- Fricción estática -->
+    <mu2>1.5</mu2>  <!-- Fricción dinámica -->
+    <kp>1e6</kp>    <!-- Rigidez del contacto -->
+    <kd>1e3</kd>    <!-- Amortiguamiento -->
+  </gazebo>
+  <gazebo reference="right_foot">
+    <mu1>1.5</mu1>
+    <mu2>1.5</mu2>
+    <kp>1e6</kp>
+    <kd>1e3</kd>
+  </gazebo>
+  <gazebo>
+    <mu1>1.5</mu1>
+    <mu2>1.5</mu2>
+    <kp>1e6</kp>
+    <kd>1e3</kd>
+  </gazebo>
 </robot>

Commit message: intentar pato parado

File: src/urdf_description/urdf/go_bdx.urdf.xacro (robot description, xacro)
@@ -72,5 +72,5 @@
     <parent link="right_hip"/>
     <child link="right_thigh"/>
-    <axis xyz="-0.0 -1.0 0.0"/>
+    <axis xyz="-0.0 1.0 0.0"/>
     <limit lower="-0.7853982" upper="0.7853982" effort="23.7" velocity="30"/>
   </joint>
@@ -79,5 +79,5 @@
     <parent link="right_thigh"/>
     <child link="right_shin"/>
-    <axis xyz="0.0 1.0 -0.0"/>
+    <axis xyz="0.0 -1.0 -0.0"/>
     <limit lower="-0.7853982" upper="0.7853982" effort="23.7" velocity="30"/>
   </joint>
@@ -86,8 +86,8 @@
     <parent link="right_shin"/>
     <child link="right_foot_link"/>
-    <axis xyz="-0.0 -1.0 0.0"/>
-    <limit lower="-0.7853982" upper="0.7853982" effort="23.7" velocity="30"/>
-  </joint>
-  <joint name="neck_pitch" type="revolute">
+    <axis xyz="-0.0 1.0 0.0"/>
+    <limit lower="-0.7853982" upper="0.7853982" effort="23.7" velocity="30"/>
+  </joint>
+  <joint name="neck_pitch" type="fixed">
     <origin rpy="0 0 0" xyz="0.056339 0.0119 0.395171"/>
     <parent link="pelvis"/>
@@ -96,5 +96,5 @@
     <limit lower="-0.7853982" upper="0.7853982" effort="23.7" velocity="30"/>
   </joint>
-  <joint name="head_pitch" type="revolute">
+  <joint name="head_pitch" type="fixed">
     <origin rpy="0 0 0" xyz="-0.065022 -0.01175 0.11088"/>
     <parent link="neck"/>
@@ -103,5 +103,5 @@
     <limit lower="-0.7853982" upper="0.7853982" effort="7.3" velocity="5.55"/>
   </joint>
-  <joint name="head_yaw" type="revolute">
+  <joint name="head_yaw" type="fixed">
     <origin rpy="0 0 0" xyz="0.000299 0.0007 0.02897"/>
     <parent link="head_body_pitch"/>
@@ -110,5 +110,5 @@
     <limit lower="-0.7853982" upper="0.7853982" effort="7.3" velocity="5.55"/>
   </joint>
-  <joint name="head_roll" type="revolute">
+  <joint name="head_roll" type="fixed">
     <origin rpy="0 0 0" xyz="0.039892 0.0 0.02715"/>
     <parent link="head_body_yaw"/>
@@ -117,5 +117,5 @@
     <limit lower="-0.7853982" upper="0.7853982" effort="7.3" velocity="5.55"/>
   </joint>
-  <joint name="left_antenna" type="revolute">
+  <joint name="left_antenna" type="fixed">
     <origin rpy="0 0 0" xyz="-0.16665 0.0683 0.001231"/>
     <parent link="head_body_roll"/>
@@ -124,5 +124,5 @@
     <limit lower="-0.7853982" upper="0.7853982" effort="0.2943" velocity="13.62"/>
   </joint>
-  <joint name="right_antenna" type="revolute">
+  <joint name="right_antenna" type="fixed">
     <origin rpy="0 0 0" xyz="-0.16665 -0.0697 0.001231"/>
     <parent link="head_body_roll"/>
@@ -514,106 +514,5 @@
     </collision>
   </link>
-  <!-- Transmissions para pierna izquierda -->
-  <transmission name="left_hip_yaw_trans">
-    <type>transmission_interface/SimpleTransmission</type>
-    <joint name="left_hip_yaw">
-      <hardwareInterface>PositionJointInterface</hardwareInterface>
-    </joint>
-    <actuator name="left_hip_yaw_motor">
-      <hardwareInterface>PositionJointInterface</hardwareInterface>
-      <mechanicalReduction>1</mechanicalReduction>
-    </actuator>
-  </transmission>
-  <transmission name="left_hip_roll_trans">
-    <type>transmission_interface/SimpleTransmission</type>
-    <joint name="left_hip_roll">
-      <hardwareInterface>PositionJointInterface</hardwareInterface>
-    </joint>
-    <actuator name="left_hip_roll_motor">
-      <hardwareInterface>PositionJointInterface</hardwareInterface>
-      <mechanicalReduction>1</mechanicalReduction>
-    </actuator>
-  </transmission>
-  <transmission name="left_hip_pitch_trans">
-    <type>transmission_interface/SimpleTransmission</type>
-    <joint name="left_hip_pitch">
-      <hardwareInterface>PositionJointInterface</hardwareInterface>
-    </joint>
-    <actuator name="left_hip_pitch_motor">
-      <hardwareInterface>PositionJointInterface</hardwareInterface>
-      <mechanicalReduction>1</mechanicalReduction>
-    </actuator>
-  </transmission>
-  <transmission name="left_knee_trans">
-    <type>transmission_interface/SimpleTransmission</type>
-    <joint name="left_knee">
-      <hardwareInterface>PositionJointInterface</hardwareInterface>
-    </joint>
-    <actuator name="left_knee_motor">
-      <hardwareInterface>PositionJointInterface</hardwareInterface>
-      <mechanicalReduction>1</mechanicalReduction>
-    </actuator>
-  </transmission>
-  <transmission name="left_ankle_trans">
-    <type>transmission_interface/SimpleTransmission</type>
-    <joint name="left_ankle">
-      <hardwareInterface>PositionJointInterface</hardwareInterface>
-    </joint>
-    <actuator name="left_ankle_motor">
-      <hardwareInterface>PositionJointInterface</hardwareInterface>
-      <mechanicalReduction>1</mechanicalReduction>
-    </actuator>
-  </transmission>
-  <!-- Transmissions para pierna derecha -->
-  <transmission name="right_hip_yaw_trans">
-    <type>transmission_interface/SimpleTransmission</type>
-    <joint name="right_hip_yaw">
-      <hardwareInterface>PositionJointInterface</hardwareInterface>
-    </joint>
-    <actuator name="right_hip_yaw_motor">
-      <hardwareInterface>PositionJointInterface</hardwareInterface>
-      <mechanicalReduction>1</mechanicalReduction>
-    </actuator>
-  </transmission>
-  <transmission name="right_hip_roll_trans">
-    <type>transmission_interface/SimpleTransmission</type>
-    <joint name="right_hip_roll">
-      <hardwareInterface>PositionJointInterface</hardwareInterface>
-    </joint>
-    <actuator name="right_hip_roll_motor">
-      <hardwareInterface>PositionJointInterface</hardwareInterface>
-      <mechanicalReduction>1</mechanicalReduction>
-    </actuator>
-  </transmission>
-  <transmission name="right_hip_pitch_trans">
-    <type>transmission_interface/SimpleTransmission</type>
-    <joint name="right_hip_pitch">
-      <hardwareInterface>PositionJointInterface</hardwareInterface>
-    </joint>
-    <actuator name="right_hip_pitch_motor">
-      <hardwareInterface>PositionJointInterface</hardwareInterface>
-      <mechanicalReduction>1</mechanicalReduction>
-    </actuator>
-  </transmission>
-  <transmission name="right_knee_trans">
-    <type>transmission_interface/SimpleTransmission</type>
-    <joint name="right_knee">
-      <hardwareInterface>PositionJointInterface</hardwareInterface>
-    </joint>
-    <actuator name="right_knee_motor">
-      <hardwareInterface>PositionJointInterface</hardwareInterface>
-      <mechanicalReduction>1</mechanicalReduction>
-    </actuator>
-  </transmission>
-  <transmission name="right_ankle_trans">
-    <type>transmission_interface/SimpleTransmission</type>
-    <joint name="right_ankle">
-      <hardwareInterface>PositionJointInterface</hardwareInterface>
-    </joint>
-    <actuator name="right_ankle_motor">
-      <hardwareInterface>PositionJointInterface</hardwareInterface>
-      <mechanicalReduction>1</mechanicalReduction>
-    </actuator>
-  </transmission>
+<!-- robot control-->
   <ros2_control name="robot_controller" type="system">
     <hardware>
@@ -738,24 +637,24 @@
     </plugin>
   </gazebo>
-  <gazebo reference="left_foot">
-    <mu1>1.5</mu1>  <!-- Fricción estática -->
-    <mu2>1.5</mu2>  <!-- Fricción dinámica -->
-    <kp>1e6</kp>    <!-- Rigidez del contacto -->
-    <kd>1e3</kd>    <!-- Amortiguamiento -->
-  </gazebo>
-  <gazebo reference="right_foot">
-    <mu1>1.5</mu1>
-    <mu2>1.5</mu2>
-    <kp>1e6</kp>
-    <kd>1e3</kd>
-  </gazebo>
-  <gazebo>
-    <mu1>1.5</mu1>
-    <mu2>1.5</mu2>
-    <kp>1e6</kp>
-    <kd>1e3</kd>
-  </gazebo>
-  <gazebo>
-    <static>true</static>
+  <gazebo reference="ear_right">
+    <gravity>0</gravity>
+  </gazebo>
+  <gazebo reference="ear_left">
+    <gravity>0</gravity>
+  </gazebo>
+  <gazebo reference="head">
+    <gravity>0</gravity>
+  </gazebo>
+  <gazebo reference="head_body_roll">
+    <gravity>0</gravity>
+  </gazebo>
+  <gazebo reference="head_body_yaw">
+    <gravity>0</gravity>
+  </gazebo>
+  <gazebo reference="head_body_pitch">
+    <gravity>0</gravity>
+  </gazebo>
+  <gazebo reference="neck">
+    <gravity>0</gravity>
   </gazebo>
 </robot>

Commit message: gazebo y rviz sincronizado, pato aun tirado y ambos doblan las patitas

File: src/urdf_description/urdf/go_bdx.urdf.xacro (robot description, xacro)
@@ -514,4 +514,107 @@
     </collision>
   </link>
+<!-- Transmissions -->
+  <!-- Transmissions para pierna izquierda -->
+  <transmission name="left_hip_yaw_trans">
+    <type>transmission_interface/SimpleTransmission</type>
+    <joint name="left_hip_yaw">
+      <hardwareInterface>position</hardwareInterface>
+    </joint>
+    <actuator name="left_hip_yaw_motor">
+      <hardwareInterface>position</hardwareInterface>
+      <mechanicalReduction>1</mechanicalReduction>
+    </actuator>
+  </transmission>
+  <transmission name="left_hip_roll_trans">
+    <type>transmission_interface/SimpleTransmission</type>
+    <joint name="left_hip_roll">
+      <hardwareInterface>position</hardwareInterface>
+    </joint>
+    <actuator name="left_hip_roll_motor">
+      <hardwareInterface>position</hardwareInterface>
+      <mechanicalReduction>1</mechanicalReduction>
+    </actuator>
+  </transmission>
+  <transmission name="left_hip_pitch_trans">
+    <type>transmission_interface/SimpleTransmission</type>
+    <joint name="left_hip_pitch">
+      <hardwareInterface>position</hardwareInterface>
+    </joint>
+    <actuator name="left_hip_pitch_motor">
+      <hardwareInterface>position</hardwareInterface>
+      <mechanicalReduction>1</mechanicalReduction>
+    </actuator>
+  </transmission>
+  <transmission name="left_knee_trans">
+    <type>transmission_interface/SimpleTransmission</type>
+    <joint name="left_knee">
+      <hardwareInterface>position</hardwareInterface>
+    </joint>
+    <actuator name="left_knee_motor">
+      <hardwareInterface>position</hardwareInterface>
+      <mechanicalReduction>1</mechanicalReduction>
+    </actuator>
+  </transmission>
+  <transmission name="left_ankle_trans">
+    <type>transmission_interface/SimpleTransmission</type>
+    <joint name="left_ankle">
+      <hardwareInterface>position</hardwareInterface>
+    </joint>
+    <actuator name="left_ankle_motor">
+      <hardwareInterface>position</hardwareInterface>
+      <mechanicalReduction>1</mechanicalReduction>
+    </actuator>
+  </transmission>
+  <!-- Transmissions para pierna derecha -->
+  <transmission name="right_hip_yaw_trans">
+    <type>transmission_interface/SimpleTransmission</type>
+    <joint name="right_hip_yaw">
+      <hardwareInterface>position</hardwareInterface>
+    </joint>
+    <actuator name="right_hip_yaw_motor">
+      <hardwareInterface>position</hardwareInterface>
+      <mechanicalReduction>1</mechanicalReduction>
+    </actuator>
+  </transmission>
+  <transmission name="right_hip_roll_trans">
+    <type>transmission_interface/SimpleTransmission</type>
+    <joint name="right_hip_roll">
+      <hardwareInterface>position</hardwareInterface>
+    </joint>
+    <actuator name="right_hip_roll_motor">
+      <hardwareInterface>position</hardwareInterface>
+      <mechanicalReduction>1</mechanicalReduction>
+    </actuator>
+  </transmission>
+  <transmission name="right_hip_pitch_trans">
+    <type>transmission_interface/SimpleTransmission</type>
+    <joint name="right_hip_pitch">
+      <hardwareInterface>position</hardwareInterface>
+    </joint>
+    <actuator name="right_hip_pitch_motor">
+      <hardwareInterface>position</hardwareInterface>
+      <mechanicalReduction>1</mechanicalReduction>
+    </actuator>
+  </transmission>
+  <transmission name="right_knee_trans">
+    <type>transmission_interface/SimpleTransmission</type>
+    <joint name="right_knee">
+      <hardwareInterface>position</hardwareInterface>
+    </joint>
+    <actuator name="right_knee_motor">
+      <hardwareInterface>position</hardwareInterface>
+      <mechanicalReduction>1</mechanicalReduction>
+    </actuator>
+  </transmission>
+  <transmission name="right_ankle_trans">
+    <type>transmission_interface/SimpleTransmission</type>
+    <joint name="right_ankle">
+      <hardwareInterface>position</hardwareInterface>
+    </joint>
+    <actuator name="right_ankle_motor">
+      <hardwareInterface>position</hardwareInterface>
+      <mechanicalReduction>1</mechanicalReduction>
+    </actuator>
+  </transmission>
 <!-- robot control-->
   <ros2_control name="robot_controller" type="system">
